File: blackbody_a/blackbody_a.kicad_sch (KiCad schematic)
At the start: 3 parts, among them J1 Conn_01x04, J2 Conn_01x04, J3 Conn_01x04

Commit message: Fixed pins, minor changes, removed power isolation
Parts:
- removed J2: Conn_01x04, symbol Connector_Generic:Conn_01x04
- added C12, C13: 12p, symbol Device:C
- added C19: 4.7uF, symbol Device:C
- added C20, C21, C22, C24: 100nF, symbol Device:C
- added C23: 100nF, Capacitor_SMD:C_0805_2012Metric, symbol Device:C
- added CAN_IN, CAN_OUT, Power: Conn_01x02, symbol Connector_Generic:Conn_01x02
- added D11: I2C, LED_SMD:LED_0805_2012Metric, symbol Device:LED
- added D12: Heartbeat, LED_SMD:LED_0805_2012Metric, symbol Device:LED
- added D8: Error, LED_SMD:LED_0805_2012Metric, symbol Device:LED
- added R17, R21, R22: 2.2k, Resistor_SMD:R_0805_2012Metric, symbol Device:R
- added R23: 10k, symbol Device:R_US
- added SW4: SW_SPDT, symbol Switch:SW_SPDT
- added SW5: SW_Push, Button_Switch_SMD:SW_SPST_B3SL-1002P, symbol Switch:SW_Push
- added SW6: Reset, symbol Switch:SW_Push
- added U3: STM32L431CBTx, Package_QFP:LQFP-48_7x7mm_P0.5mm, symbol MCU_ST_STM32L4:STM32L431CBTx
- added Y1: 8M, symbol Device:Crystal
- renumbered J1 to BlackbodyC, J3 to SWD
Connections:
- net +3V3: now also C19.1, C20.1, C21.1, C22.1, R23.1, U3.24 (VDD), U3.36 (VDD), U3.48 (VDD), U3.9 (VDDA)
- net 12V_Ext: now also Power.1 (Pin_1)
- net CAN_H: now also CAN_IN.2 (Pin_2), CAN_OUT.2 (Pin_2)
- net CAN_L: now also CAN_IN.1 (Pin_1), CAN_OUT.1 (Pin_1)
- net GND: now also C12.1, C13.1, C19.2, C20.2, C21.2, C22.2, C23.2, C24.1, D11.1 (K), D12.1 (K), D8.1 (K), Power.2 (Pin_2), SW4.3 (C), SW5.1, SW6.2, U3.23 (VSS), U3.35 (VSS), U3.44 (PH3), U3.47 (VSS), U3.8 (VSSA)
- net SWCLK: now also U3.37 (PA14)
- net SWDIO: now also U3.34 (PA13)
- new net: C13.2, U3.6 (PH1), Y1.2
- new net: D8.2 (A), R17.2
- new net: D11.2 (A), R21.2
- new net: D12.2 (A), R22.2
- new net: C12.2, U3.5 (PH0), Y1.1
- new net CAN_RX: U3.32 (PA11)
- new net CAN_TX: U3.33 (PA12)
- new net Error: R17.1, U3.11 (PA1)
- new net Heartbeat: R22.1, U3.10 (PA0)
- new net I2C: R21.1, U3.12 (PA2)
- new net I2C1_SCL: U3.42 (PB6)
- new net I2C1_SDA: U3.43 (PB7)
- new net NRST: C24.2, R23.2, SW6.1, U3.7 (NRST)
- new net SW_PUSH: C23.1, SW5.2, U3.14 (PA4)
- new net SW_SLIDE: SW4.2 (B), U3.13 (PA3)
- no-connect marks 0 -> 26
Other:
- removed sheet controller
- sheet can_comm ports: added none; removed 3V3_bus
- sheet power_dist ports: added none; removed 3V3_bus
- note added: "Bypass Capacitors"
- note added: "Controller"
- note added: "LEDs"
- note added: "Reset Button"
- moved on the sheet: BlackbodyC, SWD

Commit message: review changes
Parts:
- removed Power: Conn_01x02, symbol Connector_Generic:Conn_01x02
- added J1: CarPowerConnector, symbol utsvt-connectors:CarPowerConnector
- added R3: 10k, symbol Device:R_US
Connections:
- net I2C1_SCL is gone; now on net SCL: U3.42 (PB6)
- net I2C1_SDA is gone; now on net SDA: U3.43 (PB7)
- net 12V_Ext: now also J1.1 (+12V)
- net GND: now also SWD.3 (Pin_3), J1.2 (GND), R3.2; no longer SWD.4 (Pin_4), U3.44 (PH3)
- net SWDIO: now also SWD.4 (Pin_4); no longer SWD.3 (Pin_3)
- new net: R3.1, U3.44 (PH3)

Commit message: layout iteration 1
Parts:
- BlackbodyC1: renamed from BlackbodyC; footprint (none) -> blackbodies:MOLEX_1053091104
- C12, C13, C19, C20, C21, C22, C24: footprint (none) -> Capacitor_SMD:C_0805_2012Metric
- CAN_IN1: renamed from CAN_IN; footprint (none) -> Connector_PinHeader_2.54mm:PinHeader_1x02_P2.54mm_Vertical
- CAN_OUT1: renamed from CAN_OUT; footprint (none) -> Connector_PinHeader_2.54mm:PinHeader_1x02_P2.54mm_Vertical
- J1: footprint (none) -> UTSVT_Connectors:Molex_MicroFit3.0_1x2xP3.00mm_PolarizingPeg_Vertical
- R23, R3: footprint (none) -> Resistor_SMD:R_0805_2012Metric
- SW4: footprint (none) -> Button_Switch_SMD:SW_DIP_SPSTx01_Slide_6.7x4.1mm_W6.73mm_P2.54mm_LowProfile_JPin
- SW6: footprint (none) -> Button_Switch_SMD:SW_SPST_B3SL-1002P
- SWD1: renamed from SWD; footprint (none) -> Connector_PinHeader_2.54mm:PinHeader_1x04_P2.54mm_Vertical
- Y1: footprint (none) -> UTSVT_Special:ABM3
Other:
- moved on the sheet: BlackbodyC1, C12, C13, C19, C20, C21, C22, CAN_IN1, CAN_OUT1, J1, R3, SWD1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

Commit message: layout edits
Parts:
- added J2: Conn_02x04_Counter_Clockwise, Connector_PinHeader_2.54mm:PinHeader_2x04_P2.54mm_Vertical, symbol Connector_Generic:Conn_02x04_Counter_Clockwise
- BlackbodyC1: footprint blackbodies:MOLEX_1053091104 -> Connector_Molex:Molex_Nano-Fit_105313-xx04_1x04_P2.50mm_Horizontal
- CAN_IN1, CAN_OUT1: footprint Connector_PinHeader_2.54mm:PinHeader_1x02_P2.54mm_Vertical -> blackbodies:CONN_SD-105309-100_02_MOL
Connections:
- net SCL: now also BlackbodyC1.1 (Pin_1); no longer BlackbodyC1.2 (Pin_2)
- net SDA: now also BlackbodyC1.2 (Pin_2); no longer BlackbodyC1.1 (Pin_1)
- net 15: now reaches U3.15 (PA5)
- net 15: now also J2.8 (Pin_8)
- net 16: now reaches U3.16 (PA6)
- net 16: now also J2.7 (Pin_7)
- net 17: now reaches U3.17 (PA7)
- net 17: now also J2.6 (Pin_6)
- net 18: now reaches U3.18 (PB0)
- net 18: now also J2.5 (Pin_5)
- net 19: now reaches U3.19 (PB1)
- net 19: now also J2.4 (Pin_4)
- net 20: now reaches U3.20 (PB2)
- net 20: now also J2.3 (Pin_3)
- net 21: now reaches U3.21 (PB10)
- net 21: now also J2.2 (Pin_2)
- net 22: now reaches U3.22 (PB11)
- net 22: now also J2.1 (Pin_1)
- net +3V3 renamed +3.3V
- no-connect marks 26 -> 18
Other:
- note added: "Breakouts"
- moved on the sheet: R3
