File: blackbody_a/power_dist.kicad_sch (KiCad schematic)
At the start: 0 parts

Commit message: Added power distribution
Parts:
- added C14, C16, C17, C19: 10uF, symbol Device:C
- added C15: 0.1uF, symbol Device:C
- added D3, D5: 12V, LED_SMD:LED_0805_2012Metric, symbol Device:LED
- added D4: 3.3V, LED_SMD:LED_0805_2012Metric, symbol Device:LED
- added IC2: TPS562231DRLR, SOTFL50P160X60-6N, symbol TPS562231DRLR:TPS562231DRLR
- added L1: 3.3uH, symbol Device:L
- added R11: 45.3k, Resistor_SMD:R_0805_2012Metric, symbol Device:R
- added R12: 10k, Resistor_SMD:R_0805_2012Metric, symbol Device:R
- added R13, R15: 22.1k, Resistor_SMD:R_0805_2012Metric, symbol Device:R
- added R14: 2.2k, Resistor_SMD:R_0805_2012Metric, symbol Device:R
- added TP1, TP2, TP3, TP4, TP5: TestPoint, symbol Connector:TestPoint
- added U4: RO-123.3S_HP, UTSVT_ICs:RI3_DC_Converter, symbol utsvt-power-regulators:RO-123.3S_HP
Connections:
- new net: D4.2 (A), R14.2
- new net: IC2.6 (FB), R11.2, R12.1
- new net: D3.2 (A), R13.2
- new net: D5.2 (A), R15.2
- new net +12V: C14.1, C16.1, C17.1, IC2.1 (VIN), IC2.5 (EN), R13.1, TP1.1, U4.2 (+Vin)
- new net +3.3V: C19.1, R14.1, U4.4 (+Vout)
- new net +3V3: TP4.1
- new net 12V_Ext: R15.1
- new net 3V3_bus: L1.2, R11.1, TP2.1
- new net BST: C15.1, IC2.4 (BST)
- new net Fault: D5.1 (K)
- new net GND: C19.2, D4.1 (K), TP5.1, U4.3 (-Vout)
- new net GNDPWR: C14.2, C16.2, C17.2, D3.1 (K), IC2.3 (GND), R12.2, TP3.1, U4.1 (-Vin)
- new net SW: C15.2, IC2.2 (SW), L1.1
Other:
- added sheet power_protection (power_protection.kicad_sch)
- note added: "Isolated 12V -> 3.3V"
- note added: "LEDs"
- note added: "Testpoints"
- note added: "Unisolated 12V -> 3.3V"
- note added: "Vin Power Protection"

Commit message: minor errors
Changed lines of the file:
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@@
+	)
+	(junction
+		(at 93.98 113.03)
+		(diameter 0)
+		(color 0 0 0 0)
 	)
 	(junction
@@
 					(unit 1)
 				)
+			)
+		)
+	)
+	(symbol
+		(lib_id "power:PWR_FLAG")
+		(at 93.98 113.03 0)
+		(unit 1)
+		(exclude_from_sim no)
+		(in_bom yes)
+		(on_board yes)
+		(dnp no)
+		(fields_autoplaced yes)
+		(property "Reference" "#FLG02"
+			(at 93.98 111.125 0)
+			(effects
+				(font
+					(size 1.27 1.27)
+				)
+				(hide yes)
+			)
+		)
+		(property "Value" "PWR_FLAG"
+			(at 93.98 107.95 0)
+			(effects
+				(font
+					(size 1.27 1.27)
+				)
+			)
+		)
+		(property "Footprint" ""
+			(at 93.98 113.03 0)
+			(effects
+				(font
+					(size 1.27 1.27)
+				)
+				(hide yes)
+			)
+		)
+		(property "Datasheet" "~"
+			(at 93.98 113.03 0)
+			(effects
+				(font
+					(size 1.27 1.27)
+				)
+				(hide yes)
+			)
+		)
+		(property "Description" "Special symbol for telling ERC where power comes from"
+			(at 93.98 113.03 0)
+			(effects
+				(font
+					(size 1.27 1.27)
+				)
+				(hide yes)
+			)
+		)
+		(pin "1"
+		)
+		(instances
+			(project "blackbody_a"
+				(path "/1fc8ae43-742a-46b6-a93b-79253d0d0202/4ab23797-193f-4d52-9392-152adca945ed"
+					(reference "#FLG02")
+					(unit 1)
+				)

Commit message: Fixed pins, minor changes, removed power isolation
Parts:
- removed C16, C17, C19: 10uF, symbol Device:C
- removed TP2, TP3: TestPoint, symbol Connector:TestPoint
- removed U4: RO-123.3S_HP, UTSVT_ICs:RI3_DC_Converter, symbol utsvt-power-regulators:RO-123.3S_HP
- added C10: 100nF, Capacitor_SMD:C_0805_2012Metric, symbol Device:C
- added C11: 47uF, symbol Device:C
- added C2, C3: 10uF, Capacitor_SMD:C_0805_2012Metric, symbol Device:C
- added D2: SD12_SOD323, Diode_SMD:D_SOD-323, symbol Diode:SD12_SOD323
- added IC1: LM76202QPWPRQ1, SOP65P640X120-17N, symbol LM76202QPWPRQ1:LM76202QPWPRQ1
- added R10, R8: 10K, Resistor_SMD:R_0805_2012Metric, symbol Device:R
- added R5: 10k, Resistor_SMD:R_0805_2012Metric, symbol Device:R
- added R6: 200, Resistor_SMD:R_0805_2012Metric, symbol Device:R
- added R7: 1k, Resistor_SMD:R_0805_2012Metric, symbol Device:R
- added R9: 100k, Resistor_SMD:R_0805_2012Metric, symbol Device:R
Connections:
- net 3V3_bus is gone; now on net +3.3V: L1.2, R11.1
- net GNDPWR is gone; now on net GND: C14.2, D3.1 (K), IC2.3 (GND), R12.2
- net +12V: now also C3.1, IC1.15 (OUT_1), IC1.16 (OUT_2), R9.1
- net +3.3V: now also C11.1, R8.1
- net 12V_Ext: now also C2.1, D2.2 (A2), IC1.1 (IN_1), IC1.2 (IN_2), R5.1
- net Fault: now also IC1.14 (~{FLT}), R9.2
- net GND: now also C11.2, C2.2, C3.2, D2.1 (A1), IC1.9 (GND)
- new net: IC1.11 (ILIM), R10.1
- new net: C10.1, IC1.12 (DVDT)
- new net: IC1.7 (~{SHDN}), R8.2
- new net OVP: IC1.5 (OVP), R6.2, R7.1
- new net RTN: C10.2, IC1.13 (NC_2), IC1.17 (EP), IC1.4 (NC_1), IC1.6 (MODE), IC1.8 (RTN), R10.2, R7.2
- new net UVLO: IC1.3 (UVLO), R5.2, R6.1
- no-connect marks 0 -> 1
Other:
- removed sheet power_protection
- note added: "12V -> 3.3V"
- note removed: "Isolated 12V -> 3.3V"
- note removed: "Unisolated 12V -> 3.3V"
- moved on the sheet: C15, D3, D4, D5, R13, R14, R15, TP1, TP4, TP5

Commit message: layout iteration 1
Parts:
- C11, C14, C15: footprint (none) -> Capacitor_SMD:C_0805_2012Metric
- IC1: footprint SOP65P640X120-17N -> blackbody_a:LM76202QPWPRQ1
- IC2: footprint SOTFL50P160X60-6N -> blackbody_a:TPS562231DRLR
- L1: footprint (none) -> Inductor_SMD:L_0805_2012Metric
- R9: value 100k -> 10k
- TP1, TP4, TP5: footprint (none) -> TestPoint:TestPoint_Pad_D1.0mm

Commit message: layout edits
Parts:
- removed C11: 47uF, Capacitor_SMD:C_0805_2012Metric, symbol Device:C
- removed C14: 10uF, Capacitor_SMD:C_0805_2012Metric, symbol Device:C
- removed C15: 0.1uF, Capacitor_SMD:C_0805_2012Metric, symbol Device:C
- removed IC2: TPS562231DRLR, blackbody_a:TPS562231DRLR, symbol TPS562231DRLR:TPS562231DRLR
- removed L1: 3.3uH, Inductor_SMD:L_0805_2012Metric, symbol Device:L
- removed R11: 45.3k, Resistor_SMD:R_0805_2012Metric, symbol Device:R
- removed R12: 10k, Resistor_SMD:R_0805_2012Metric, symbol Device:R
- removed R6: 200, Resistor_SMD:R_0805_2012Metric, symbol Device:R
- removed R7: 1k, Resistor_SMD:R_0805_2012Metric, symbol Device:R
- added C16: 10uF, Capacitor_SMD:C_0805_2012Metric, symbol Device:C
- added C17: 0.1uF, Capacitor_SMD:C_0805_2012Metric, symbol Device:C
- added C18: 10nF, Capacitor_SMD:C_0805_2012Metric, symbol Device:C
- added C25: 4.7nF, Capacitor_SMD:C_0805_2012Metric, symbol Device:C
- added C4: 33uF, Capacitor_SMD:C_0805_2012Metric, symbol Device:C_Polarized_US
- added D6: D, Diode_SMD:D_0805_2012Metric, symbol Device:D
- added H1, H2, H3, H4: MountingHole, MountingHole:MountingHole_3.2mm_M3, symbol Mechanical:MountingHole
- added L2: 13.3uH, Inductor_SMD:L_0805_2012Metric, symbol Device:L
- added Rosc1: 85.5k, Resistor_SMD:R_0805_2012Metric, symbol Device:R
- added U4: TPS5403DR, blackbodies:D0008A_N, symbol 2025-04-15_23-22-41:TPS5403DR
- R10: value 10K -> 20K
- R5: value 10k -> 12k; Mouser Part Number 71-CRCW080510K0FKEAC -> (none); P/N CRCW08051K00FKEAC -> (none)
Connections:
- net +3V3 is gone; now on net +3.3V: TP4.1
- net +12V: now also C16.2, U4.2 (VIN)
- net +3.3V: now also C4.1, L2.2, U4.5 (VSENSE)
- net 12V_Ext: no longer R5.1
- net GND: now also C16.1, C18.2, C25.1, C4.2, D6.2 (A), Rosc1.2, U4.7 (GND)
- net RTN: no longer IC1.13 (NC_2), IC1.4 (NC_1), IC1.6 (MODE)
- net UVLO: no longer R5.2
- new net: C17.2, D6.1 (K), L2.1, U4.8 (LX)
- new net: C17.1, U4.1 (BOOT)
- new net: Rosc1.1, U4.3 (ROSC)
- new net: C18.1, U4.4 (SS)
- new net: R5.1, U4.6 (COMP)
- new net: C25.2, R5.2
- new net MODE: IC1.6 (MODE)
- no-connect marks 1 -> 3
Other:
- note added: "12V -> 3.3"
- note removed: "12V -> 3.3V"

Commit message: layout updates
Parts:
- removed L2: 13.3uH, Inductor_SMD:L_0805_2012Metric, symbol Device:L
- added L1: MSS1038-153MLC, blackbody_a:INDPM102100X400N, symbol MSS1038-153MLC:MSS1038-153MLC
- added Rosc2: 1k, Resistor_SMD:R_0805_2012Metric, symbol Device:R
- C10: Manufacturer_Part_Number (none) -> 80-C0805C104M5RACTU; Mouser Part Number 80-C0805C104M5R -> 80-C0805C104M5RACTU; PN (none) -> C0805C104M5RACTU
- C16: Manufacturer_Part_Number (none) -> TMK212BBJ106MGHT; Mouser Part Number (none) -> 963-TMK212BBJ106MGHT; PN (none) -> TMK212BBJ106MGHT
- C17: Manufacturer_Part_Number (none) -> C0805C104M5R; Mouser Part Number (none) -> 80-C0805C104M5R; PN (none) -> C0805C104M5RACTU
- C18: value 10nF -> 15nF; Manufacturer_Part_Number (none) -> C0805C104J5RACTU; Mouser Part Number (none) -> 80-C0805C104J5RACTU; PN (none) -> C0805C103J5RACTU
- C2, C3: Manufacturer_Part_Number (none) -> TMK212BBJ106MGHT; Mouser Part Number 581-22201C106KAT2A -> 963-TMK212BBJ106MGHT; PN (none) -> TMK212BBJ106MGHT
- C25: value 4.7nF -> 1nF; PN (none) -> C0805C102K5RACAUTO
- C4: value 33uF -> 22uF; PN (none) -> C0805C226M9PACTU
- D2: Manufacturer_Part_Number (none) -> PESD15VL1BA-T/R; Mouser Part Number 771-PESD15VL1BA-T/R -> 821-BZT52C12S; PN (none) -> BZT52C12S
- D3, D4, D5: Manufacturer_Part_Number (none) -> 604-APTD2012LCGCK; PN (none) -> APTD2012LCGCK
- D6: footprint Diode_SMD:D_0805_2012Metric -> blackbodies:SMA_DIO; PN (none) -> B230A13F
- IC1: PN (none) -> LM76202QPWPRQ1
- R10, R13, R15: PN (none) -> CRCW080520K0FKEA
- R14: Mouser Part Number Inventory -> 71-CRCW0805-2.2K-E3; PN (none) -> CRCW08052K20FKEA
- R5: value 12k -> 10k; Mouser Part Number (none) -> 603-RT0805FRE0710KL; PN (none) -> CRCW080510K0FKEA
- R8: PN (none) -> RT0805FRE0710KL
- R9: Mouser Part Number 71-CRCW0805100KFKEAC -> 603-RT0805FRE0710KL; PN (none) -> CRCW080510K0FKEA
- Rosc1: value 85.5k -> 84.5k; Mouser Part Number (none) -> 71-CRCW0805-84.5K-E3; PN (none) -> CRCW080584K5FKEA
- U4: Mouser Part Number (none) -> 595-TPS54233D; PN (none) -> TPS54233D
Connections:
- net +3.3V: now also L1.2
- net GND: now also Rosc2.2; no longer Rosc1.2
- net at C17.2, D6.1 (K), U4.8 (LX): now also L1.1
- new net: Rosc1.2, Rosc2.1
Other:
- moved on the sheet: C4, D6
