File: sensor_board/sensor_board.kicad_sch (KiCad schematic)
At the start: 4 parts, among them J1 Conn_01x04_Pin, U1 TSL25911FN

Commit message: Fixed pins, minor changes, removed power isolation
Parts:
- removed J1: Conn_01x04_Pin, symbol Connector:Conn_01x04_Pin
- added BlackbodyC: Conn_01x04, symbol Connector_Generic:Conn_01x04
Connections:
- net +3V3: now also BlackbodyC.3 (Pin_3)
- net GND: now also BlackbodyC.4 (Pin_4)
- net SCL: now also BlackbodyC.1 (Pin_1)
- net SDA: now also BlackbodyC.2 (Pin_2)
Other:
- moved on the sheet: C4

Commit message: layout iteration 1
Parts:
- BlackbodyC1: renamed from BlackbodyC; footprint (none) -> blackbodies:CONN_SD-105310-100_04_MOL
- C4: footprint (none) -> Capacitor_SMD:C_0402_1005Metric
- R1: footprint (none) -> Resistor_SMD:R_0402_1005Metric
- U1: footprint SON-06-FN_2000X2400_AMS -> .pretty:SON-06-FN_2000X2400_AMS
Connections:
- net SCL: now also BlackbodyC1.2 (Pin_2); no longer BlackbodyC1.1 (Pin_1)
- net SDA: now also BlackbodyC1.1 (Pin_1); no longer BlackbodyC1.2 (Pin_2)
Changed lines of the file:
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@@
 (kicad_sch
-	(version 20231120)
+	(version 20250114)
 	(generator "eeschema")
-	(generator_version "8.0")
+	(generator_version "9.0")
 	(paper "A4")
+	(text_box "Connects to blackbody c, nanofit\n"
+		(exclude_from_sim no)
+		(at 134.62 113.03 0)
+		(size 13.97 6.35)
+		(margins 0.762 0.762 0.762 0.762)
+		(stroke
+			(width 0)
+			(type default)
+		)
+		(fill
+			(type none)
+		)
+		(effects
+			(font
+				(size 1.016 1.016)
+			)
+			(justify left top)
+		)
+	)
 	(junction
 		(at 147.32 99.06)
@@
 		)
 	)
-	(text_box "Connects to blackbody c, nanofit\n"
-		(exclude_from_sim no)
-		(at 134.62 113.03 0)
-		(size 13.97 6.35)
-		(stroke
-			(width 0)
-			(type default)
-		)
-		(fill
-			(type none)
-		)
-		(effects
-			(font
-				(size 1.016 1.016)
-			)
-			(justify left top)
-		)
-	)
-	(label "SCL"
+	(label "SDA"
 		(at 107.95 111.76 0)
-		(fields_autoplaced yes)
 		(effects
 			(font
@@
 	(label "SDA"
 		(at 139.7 87.63 0)
-		(fields_autoplaced yes)
 		(effects
 			(font
@@
 		)
 	)
-	(label "SDA"
+	(label "SCL"
 		(at 107.95 114.3 0)
-		(fields_autoplaced yes)
 		(effects
 			(font
@@
 	(label "SCL"
 		(at 99.06 87.63 180)
-		(fields_autoplaced yes)
 		(effects
 			(font
@@
 			)
 		)
-		(property "Footprint" ""
+		(property "Footprint" "Capacitor_SMD:C_0402_1005Metric"
 			(at 146.3548 90.17 0)
 			(effects
@@
 			)
 		)
-		(property "Footprint" ""
+		(property "Footprint" "Resistor_SMD:R_0402_1005Metric"
 			(at 88.646 85.344 90)
 			(effects
@@
 		(dnp no)
 		(fields_autoplaced yes)
-		(property "Reference" "BlackbodyC"
+		(property "Reference" "BlackbodyC1"
 			(at 120.65 114.2999 0)
 			(effects
@@
 			)
 		)
-		(property "Footprint" ""
+		(property "Footprint" "blackbodies:CONN_SD-105310-100_04_MOL"
 			(at 118.11 114.3 0)
 			(effects
@@
 			(project "sensor_board"
 				(path "/bcce3edf-0fa4-4326-9990-2be95d501905"
-					(reference "BlackbodyC")
+					(reference "BlackbodyC1")
 					(unit 1)
 				)
@@
 			)
 		)
-		(property "Footprint" "SON-06-FN_2000X2400_AMS"
+		(property "Footprint" ".pretty:SON-06-FN_2000X2400_AMS"
 			(at 99.06 87.63 0)
 			(effects
@@
 		)
 	)
+	(embedded_fonts no)
 )

Commit message: layout edits
Parts:
- BlackbodyC1: footprint blackbodies:CONN_SD-105310-100_04_MOL -> blackbodies:CONN_SD-105429-001_04_MOL
Connections:
- net +3V3: now also BlackbodyC1.4 (Pin_4); no longer BlackbodyC1.3 (Pin_3)
- net GND: now also BlackbodyC1.3 (Pin_3); no longer BlackbodyC1.4 (Pin_4)
- net SCL: now also BlackbodyC1.1 (Pin_1); no longer BlackbodyC1.2 (Pin_2)
- net SDA: now also BlackbodyC1.2 (Pin_2); no longer BlackbodyC1.1 (Pin_1)
Changed lines of the file:
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@@
+	)
+	(junction
+		(at 104.14 119.38)
+		(diameter 0)
+		(color 0 0 0 0)
 	)
 	(junction
@@
 		(color 0 0 0 0)
 	)
-	(junction
-		(at 99.06 119.38)
-		(diameter 0)
-		(color 0 0 0 0)
-	)
 	(wire
 		(pts
@@
 	(wire
 		(pts
-			(xy 99.06 115.57) (xy 99.06 116.84)
-		)
-		(stroke
-			(width 0)
-			(type default)
-		)
-	)
-	(wire
-		(pts
 			(xy 99.06 99.06) (xy 147.32 99.06)
 		)
@@
 	(wire
 		(pts
+			(xy 104.14 119.38) (xy 113.03 119.38)
+		)
+		(stroke
+			(width 0)
+			(type default)
+		)
+	)
+	(wire
+		(pts
+			(xy 87.63 88.9) (xy 87.63 90.17)
+		)
+		(stroke
+			(width 0)
+			(type default)
+		)
+	)
+	(wire
+		(pts
 			(xy 92.71 116.84) (xy 99.06 116.84)
 		)
@@
 	(wire
 		(pts
-			(xy 87.63 88.9) (xy 87.63 90.17)
+			(xy 158.75 100.33) (xy 158.75 99.06)
+		)
+		(stroke
+			(width 0)
+			(type default)
+		)
+	)
+	(wire
+		(pts
+			(xy 99.06 92.71) (xy 99.06 99.06)
 		)
 		(stroke
@@
 	(wire
 		(pts
-			(xy 158.75 100.33) (xy 158.75 99.06)
-		)
-		(stroke
-			(width 0)
-			(type default)
-		)
-	)
-	(wire
-		(pts
-			(xy 99.06 92.71) (xy 99.06 99.06)
-		)
-		(stroke
-			(width 0)
-			(type default)
-		)
-	)
-	(wire
-		(pts
 			(xy 139.7 90.17) (xy 147.32 90.17)
 		)
@@
 	(wire
 		(pts
-			(xy 99.06 119.38) (xy 113.03 119.38)
-		)
-		(stroke
-			(width 0)
-			(type default)
-		)
-	)
-	(wire
-		(pts
-			(xy 99.06 119.38) (xy 99.06 120.65)
+			(xy 92.71 119.38) (xy 104.14 119.38)
 		)
 		(stroke
@@
 	(wire
 		(pts
+			(xy 104.14 113.03) (xy 104.14 119.38)
+		)
+		(stroke
+			(width 0)
+			(type default)
+		)
+	)
+	(wire
+		(pts
 			(xy 147.32 99.06) (xy 158.75 99.06)
 		)
@@
 	(wire
 		(pts
-			(xy 92.71 119.38) (xy 99.06 119.38)
+			(xy 99.06 116.84) (xy 99.06 120.65)
 		)
 		(stroke
@@
 		)
 	)
-	(label "SDA"
+	(label "SCL"
 		(at 107.95 111.76 0)
 		(effects
@@
 		)
 	)
-	(label "SCL"
+	(label "SDA"
 		(at 107.95 114.3 0)
 		(effects
@@
 	(symbol
 		(lib_id "power:+3V3")
-		(at 99.06 115.57 0)
-		(unit 1)
-		(exclude_from_sim no)
-		(in_bom yes)
-		(on_board yes)
-		(dnp no)
-		(fields_autoplaced yes)
-		(property "Reference" "#PWR01"
-			(at 99.06 119.38 0)
-			(effects
-				(font
-					(size 1.27 1.27)
-				)
-				(hide yes)
-			)
-		)
-		(property "Value" "+3V3"
-			(at 99.06 110.49 0)
-			(effects
-				(font
-					(size 1.27 1.27)
-				)
-			)
-		)
-		(property "Footprint" ""
-			(at 99.06 115.57 0)
-			(effects
-				(font
-					(size 1.27 1.27)
-				)
-				(hide yes)
-			)
-		)
-		(property "Datasheet" ""
-			(at 99.06 115.57 0)
-			(effects
-				(font
-					(size 1.27 1.27)
-				)
-				(hide yes)
-			)
-		)
-		(property "Description" "Power symbol creates a global label with name \"+3V3\""
-			(at 99.06 115.57 0)
-			(effects
-				(font
-					(size 1.27 1.27)
-				)
-				(hide yes)
-			)
-		)
-		(pin "1"
-		)
-		(instances
-			(project "sensor_board"
-				(path "/bcce3edf-0fa4-4326-9990-2be95d501905"
-					(reference "#PWR01")
-					(unit 1)
-				)
-			)
-		)
-	)
-	(symbol
-		(lib_id "power:+3V3")
 		(at 87.63 81.28 0)
 		(unit 1)
@@
 			)
 		)
-		(property "Footprint" "blackbodies:CONN_SD-105310-100_04_MOL"
+		(property "Footprint" "blackbodies:CONN_SD-105429-001_04_MOL"
 			(at 118.11 114.3 0)
 			(effects
@@
 					(unit 1)
 				)
+			)
+		)
+	)
+	(symbol
+		(lib_id "power:+3V3")
+		(at 104.14 113.03 0)
+		(unit 1)
+		(exclude_from_sim no)
+		(in_bom yes)
+		(on_board yes)
+		(dnp no)
+		(fields_autoplaced yes)
+		(property "Reference" "#PWR05"
+			(at 104.14 116.84 0)
+			(effects
+				(font
+					(size 1.27 1.27)
+				)
+				(hide yes)
+			)
+		)
+		(property "Value" "+3V3"
+			(at 104.14 107.95 0)
+			(effects
+				(font
+					(size 1.27 1.27)
+				)
+			)
+		)
+		(property "Footprint" ""
+			(at 104.14 113.03 0)
+			(effects
+				(font
+					(size 1.27 1.27)
+				)
+				(hide yes)
+			)
+		)
+		(property "Datasheet" ""
+			(at 104.14 113.03 0)
+			(effects
+				(font
+					(size 1.27 1.27)
+				)
+				(hide yes)
+			)
+		)
+		(property "Description" "Power symbol creates a global label with name \"+3V3\""
+			(at 104.14 113.03 0)
+			(effects
+				(font
+					(size 1.27 1.27)
+				)
+				(hide yes)
+			)
+		)
+		(pin "1"
+		)
+		(instances
+			(project "sensor_board"
+				(path "/bcce3edf-0fa4-4326-9990-2be95d501905"
+					(reference "#PWR05")
+					(unit 1)
+				)

Commit message: layout updates
Parts:
- added Power1: D, LED_SMD:LED_0805_2012Metric, symbol Device:D
- added R2: 2k, Resistor_SMD:R_0805_2012Metric, symbol Device:R_US
- BlackbodyC1: PN (none) -> 105405-2204
- C4: footprint Capacitor_SMD:C_0402_1005Metric -> Capacitor_SMD:C_0805_2012Metric; PN (none) -> C0805C105K5PACTU
- R1: footprint Resistor_SMD:R_0402_1005Metric -> Resistor_SMD:R_0805_2012Metric; PN (none) -> CRCW08051K00FKEAC
- U1: PN (none) -> TSL25911FN
Connections:
- net +3V3: now also R2.1
- net GND: now also Power1.1 (K)
- new net: Power1.2 (A), R2.2
