File: _autosave-Black Body A.kicad_sch (KiCad schematic)
At the start: 8 parts, among them IC1 MCP96L00T-E_MX, J1 Conn_01x02_Pin, J2 53307-2471, U1 TSL25911FN

Commit message: Layout Added
Parts:
- removed C1: 1uF, symbol Device:C
- removed IC1: MCP96L00T-E_MX, QFN65P500X500X100-21N-D, symbol SamacSys_Parts:MCP96L00T-E_MX
- removed J1: Conn_01x02_Pin, symbol Connector:Conn_01x02_Pin
- removed J2: 53307-2471, UTSVT_Connectors:PeripheralSOM, symbol UTSVT Connectors:PeripheralSOMConnector
- removed R1, R2: Rp, symbol Device:R_US
- removed R3: Rpi, symbol Device:R_US
- removed U1: TSL25911FN, OptoDevice:AMS_TSL25911FN, symbol Sensor_Optical:TSL25911FN
- added C2: 1uF, Capacitor_SMD:C_0603_1608Metric_Pad1.08x0.95mm_HandSolder, symbol Device:C
- added C3: 0.1u, Capacitor_SMD:C_0603_1608Metric_Pad1.08x0.95mm_HandSolder, symbol Device:C
- added D1, D2, D3, D4: 3V3, Diode_SMD:D_0603_1608Metric_Pad1.05x0.95mm_HandSolder, symbol Device:D
- added FB1, FB2: 200, Inductor_SMD:L_0603_1608Metric_Pad1.05x0.95mm_HandSolder, symbol Device:FerriteBead
- added IC2: MCP96L00T-E_MX, Blackbody Footprint:QFN65P500X500X100-21N-D, symbol Blackbody Symbols:MCP96L00T-E_MX
- added J1: 53307-2471, UTSVT_Connectors:PeripheralSOM, symbol UTSVT Connectors:PeripheralSOMConnector
- added J2: Conn_01x02, Connector_Molex:Molex_Nano-Fit_105313-xx02_1x02_P2.50mm_Horizontal, symbol Connector_Generic:Conn_01x02
- added J3: Conn_01x03, Connector_Molex:Molex_Nano-Fit_105313-xx03_1x03_P2.50mm_Horizontal, symbol Connector_Generic:Conn_01x03
- added J4: Conn_02x08_Top_Bottom, MX150:CONN_SD-75900-001_2X08_MOL, symbol Connector_Generic:Conn_02x08_Top_Bottom
- added R4: 1M, Resistor_SMD:R_0603_1608Metric_Pad0.98x0.95mm_HandSolder, symbol Device:R_US
- added R5, R6: 100, Resistor_SMD:R_0603_1608Metric_Pad0.98x0.95mm_HandSolder, symbol Device:R_US
- added R7, R8: 2M, Resistor_SMD:R_0603_1608Metric_Pad0.98x0.95mm_HandSolder, symbol Device:R_US
- added Ra1: 10k, Resistor_SMD:R_0603_1608Metric_Pad0.98x0.95mm_HandSolder, symbol Device:R_US
- added Rb1: 43k, Resistor_SMD:R_0603_1608Metric_Pad0.98x0.95mm_HandSolder, symbol Device:R_US
Connections:
- net GND: now also C2.2, D3.2 (A), D4.2 (A), IC2.1 (GND_1), IC2.10 (GND_8), IC2.13 (GND_9), IC2.17 (GND_10), IC2.18 (GND_11), IC2.21 (EPAD), IC2.3 (GND_2), IC2.5 (GND_3), IC2.6 (GND_4), IC2.7 (GND_5), IC2.9 (GND_7), J1.1 (GND), J1.3 (GND), J1.5 (GND), J4.16 (Pin_16), R7.1, R8.1, Rb1.1
- new net: FB1.1, J2.1 (Pin_1)
- new net: D1.2 (A), D3.1 (K), FB1.2, R5.2, R7.2
- new net: C3.1, IC2.2 (VIN+), R6.1
- new net: D2.2 (A), D4.1 (K), FB2.2, R4.1, R6.2, R8.2
- new net: IC2.16 (ADDR), Ra1.1, Rb1.2
- new net: C3.2, IC2.4 (VIN-), R5.1
- new net: IC2.19 (SCL), J1.6 (I2C1_SCL), J3.1 (Pin_1)
- new net: IC2.20 (SDA), J1.4 (I2C1_SDA), J3.2 (Pin_2)
- new net: J1.9 (ADC1_IN7), J3.3 (Pin_3)
- new net: FB2.1, J2.2 (Pin_2)
- new net: J1.20 (CAN_L), J4.6 (Pin_6)
- new net: J1.22 (CAN_H), J4.5 (Pin_5)
- new net: J1.24 (+24V_In), J4.1 (Pin_1)
- new net +3V3: C2.1, D1.1 (K), D2.1 (K), IC2.8 (GND_6), J1.2 (+3.3v), R4.2, Ra1.2
- no-connect marks 0 -> 34
