File: Black Body Irradiance Sensor Breakout/Black Body Breakout Board.kicad_pcb (KiCad board)
At the start: 2 copper layers, 14.9 x 13 mm, 6 parts, among them J2 Conn_01x05, U1 TSL25911FN

Commit message: updated BOM
Parts:
- moved U1 0.50 mm to (126.4, 72.7)
Routing:
- net Net-(J2-Pin_3): track 11.8 -> 10.3 mm
- net GND: track 10.9 -> 10.3 mm
Other:
- board size 14.9 x 13 mm -> 15 x 13 mm
Changed lines of the file:
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@@
 	(footprint "OptoDevice:AMS_TSL25911FN"
 		(layer "F.Cu")
-		(at 126.4625 73.2)
+		(at 126.4375 72.7)
 		(descr "DFN, 6 Pin (https://ams.com/documents/20143/9331680/TSL2591_DS000338_7-00.pdf), generated with kicad-footprint-generator ipc_noLead_generator.py")
 		(tags "DFN NoLead")
 		(property "Reference" "U1"
-			(at -0.2375 1.95 0)
+			(at 0.0625 2.3 0)
 			(layer "F.SilkS")
 			(effects
@@
 		)
 		(embedded_fonts no)
-		(model "${KICAD9_3DMODEL_DIR}/Connector_Molex.3dshapes/Molex_Nano-Fit_105313-xx05_1x05_P2.50mm_Horizontal.step"
+		(model "${KICAD9_3DMODEL_DIR}/1053131205.stp"
 			(offset
-				(xyz 0 0 0)
+				(xyz 0 -5 0)
 			)
 			(scale
@@
 			)
 			(rotate
-				(xyz 0 0 0)
-			)
-		)
-	)
-	(gr_arc
-		(start 120.796673 66.40099)
-		(mid 120.975 65.975)
-		(end 121.401878 65.798806)
+				(xyz -0 -0 -90)
+			)
+		)
+	)
+	(gr_line
+		(start 120.75 78.75)
+		(end 120.75 65.75)
 		(stroke
 			(width 0.05)
@@
 		(layer "Edge.Cuts")
 	)
-	(gr_arc
-		(start 135.122816 65.794795)
-		(mid 135.548806 65.973122)
-		(end 135.725 66.4)
+	(gr_line
+		(start 135.75 78.75)
+		(end 120.75 78.75)
 		(stroke
 			(width 0.05)
@@
 		(layer "Edge.Cuts")
 	)
-	(gr_arc
-		(start 121.4 78.775)
-		(mid 120.97401 78.596673)
-		(end 120.797816 78.169795)
+	(gr_line
+		(start 135.75 65.75)
+		(end 135.75 78.75)
 		(stroke
 			(width 0.05)
@@
 	)
 	(gr_line
-		(start 121.40591 78.775)
-		(end 135.130058 78.776194)
+		(start 120.75 65.75)
+		(end 135.75 65.75)
 		(stroke
 			(width 0.05)
@@
 		(layer "Edge.Cuts")
 	)
-	(gr_line
-		(start 121.394942 65.798806)
-		(end 135.122816 65.794795)
-		(stroke
-			(width 0.05)
-			(type default)
-		)
-		(layer "Edge.Cuts")
-	)
-	(gr_line
-		(start 135.725 66.403811)
-		(end 135.728327 78.16809)
-		(stroke
-			(width 0.05)
-			(type default)
-		)
-		(layer "Edge.Cuts")
-	)
-	(gr_line
-		(start 120.796673 66.40691)
-		(end 120.797816 78.175076)
-		(stroke
-			(width 0.05)
-			(type default)
-		)
-		(layer "Edge.Cuts")
-	)
-	(gr_arc
-		(start 135.728327 78.17401)
-		(mid 135.55 78.6)
-		(end 135.123122 78.776194)
-		(stroke
-			(width 0.05)
-			(type default)
-		)
-		(layer "Edge.Cuts")
-	)
 	(segment
 		(start 128.75 71.5)
@@
 	)
 	(segment
-		(start 128.2 73.2)
-		(end 128.25 73.25)
+		(start 127.994246 72.442719)
+		(end 127.957281 72.442719)
 		(width 0.2)
 		(layer "F.Cu")
@@
 	)
 	(segment
-		(start 127.1 73.2)
-		(end 128.2 73.2)
+		(start 127.7 72.7)
+		(end 127.075 72.7)
+		(width 0.2)
+		(layer "F.Cu")
+		(net 1)
+	)
+	(segment
+		(start 127.825763 72.574237)
+		(end 128.125764 72.574237)
+		(width 0.2)
+		(layer "F.Cu")
+		(net 1)
+	)
+	(segment
+		(start 127.7 72.7)
+		(end 127.825763 72.574237)
+		(width 0.2)
+		(layer "F.Cu")
+		(net 1)
+	)
+	(segment
+		(start 128.125764 72.574237)
+		(end 127.994246 72.442719)
 		(width 0.2)
 		(layer "F.Cu")
@@
 	)
 	(via
-		(at 128.25 73.25)
+		(at 128.125764 72.574237)
 		(size 0.6)
 		(drill 0.3)
@@
 	)
 	(segment
-		(start 128.25 72)
+		(start 128.125764 72.124236)
 		(end 128.75 71.5)
 		(width 0.2)
@@
 	)
 	(segment
-		(start 128.25 73.25)
-		(end 128.25 72)
+		(start 128.125764 72.574237)
+		(end 128.125764 72.124236)
 		(width 0.2)
 		(layer "B.Cu")
@@
 	)
 	(segment
-		(start 126.975 75)
-		(end 127.5 75)
+		(start 127.575 74.4)
+		(end 127.175 74.4)
+		(width 0.2)
+		(layer "F.Cu")
+		(net 2)
+	)
+	(segment
+		(start 126.85 74.4)
+		(end 127.175 74.4)
 		(width 0.2)
 		(layer "F.Cu")
@@
 	)
 	(segment
-		(start 125.825 73.85)
-		(end 126.975 75)
+		(start 125.8 73.35)
+		(end 126.85 74.4)
 		(width 0.2)
 		(layer "F.Cu")
@@
 	)
 	(via
-		(at 127.5 75)
+		(at 127.575 74.4)
 		(size 0.6)
 		(drill 0.3)
@@
 	)
 	(segment
+		(start 127.575 74.4)
+		(end 129.1 74.4)
+		(width 0.2)
+		(layer "B.Cu")
+		(net 2)
+	)
+	(segment
 		(start 133.25 76.93)
 		(end 133.25 76.7)
@@
 	)
 	(segment
-		(start 129 75)
-		(end 130.025 73.975)
+		(start 133.25 76.7)
+		(end 130.025 73.475)
 		(width 0.2)
 		(layer "B.Cu")
@@
 	)
 	(segment
-		(start 133.25 76.7)
+		(start 129.1 74.4)
 		(end 130.025 73.475)
 		(width 0.2)
@@
 	)
 	(segment
-		(start 130.025 73.975)
-		(end 130.025 73.475)
-		(width 0.2)
-		(layer "B.Cu")
-		(net 2)
-	)
-	(segment
-		(start 127.5 75)
-		(end 129 75)
-		(width 0.2)
-		(layer "B.Cu")
-		(net 2)
-	)
-	(segment
-		(start 125 72.5)
-		(end 125.775 72.5)
+		(start 124.675 72.25)
+		(end 124.875 72.05)
 		(width 0.2)
 		(layer "F.Cu")
@@
 	)
 	(segment
-		(start 125.825 72.55)
-		(end 125.6 72.325)
+		(start 125.6 70.4625)
+		(end 125.6 71.85)
 		(width 0.2)
 		(layer "F.Cu")
@@
 	)
 	(segment
-		(start 125.775 72.5)
-		(end 125.825 72.55)
+		(start 124.875 72.05)
+		(end 125.8 72.05)
 		(width 0.2)
 		(layer "F.Cu")
@@
 	)
 	(segment
-		(start 125.6 72.325)
-		(end 125.6 70.4625)
+		(start 125.6 71.85)
+		(end 125.8 72.05)
 		(width 0.2)
 		(layer "F.Cu")
@@
 	)
 	(via
-		(at 125 72.5)
+		(at 124.675 72.25)
 		(size 0.6)
 		(drill 0.3)
@@
 	)
 	(segment
-		(start 124.5 74)
-		(end 124.5 73)
+		(start 124.5 72.425)
+		(end 124.5 74)
 		(width 0.2)
 		(layer "B.Cu")
@@
 	)
 	(segment
-		(start 124.5 73)
-		(end 125 72.5)
+		(start 124.675 72.25)
+		(end 124.5 72.425)
 		(width 0.2)
 		(layer "B.Cu")
@@
 	)
 	(segment
-		(start 123.7125 73.2)
-		(end 125.825 73.2)
+		(start 123.7 73.9125)
+		(end 124.7635 72.849)
 		(width 0.2)
 		(layer "F.Cu")
@@
 	)
 	(segment
+		(start 125.651 72.849)
+		(end 125.8 72.7)
+		(width 0.2)
+		(layer "F.Cu")
+		(net 5)
+	)
+	(segment
 		(start 123 73.9125)
-		(end 123.7125 73.2)
+		(end 123.7 73.9125)
+		(width 0.2)
+		(layer "F.Cu")
+		(net 5)
+	)
+	(segment
+		(start 124.7635 72.849)
+		(end 125.651 72.849)
 		(width 0.2)
 		(layer "F.Cu")
@@
 	)
 	(segment
-		(start 128.851 76.679)
-		(end 128.851 72.450943)
+		(start 128.851 72.450944)
+		(end 128.0875 71.687444)
 		(width 0.2)
 		(layer "F.Cu")
@@
 	)
 	(segment
-		(start 128.45 77.08)
-		(end 127.8385 76.4685)
+		(start 128.0875 71.275)
+		(end 128.0875 69.5)
 		(width 0.2)
 		(layer "F.Cu")
@@
 	)
 	(segment
-		(start 127.1 72.55)
-		(end 127.1 71.2875)
+		(start 127.8385 76.4685)
+		(end 128.45 77.08)
 		(width 0.2)
 		(layer "F.Cu")
@@
 	)
 	(segment
-		(start 127.1 71.2875)
-		(end 128.2375 70.15)
-		(width 0.2)
-		(layer "F.Cu")
-		(net 6)
-	)
-	(segment
-		(start 128.0875 71.687443)
-		(end 128.0875 69.5)
-		(width 0.2)
-		(layer "F.Cu")
-		(net 6)
-	)
-	(segment
-		(start 128.851 72.450943)
-		(end 128.0875 71.687443)
+		(start 127.075 72.05)
+		(end 127.85 71.275)
 		(width 0.2)
 		(layer "F.Cu")
@@
 		(width 0.2)
 		(layer "F.Cu")
+		(net 6)
+	)
+	(segment
+		(start 127.85 71.275)
+		(end 128.0875 71.275)
+		(width 0.2)
+		(layer "F.Cu")
+		(net 6)
+	)
+	(segment
+		(start 128.0875 71.687444)
+		(end 128.0875 71.275)
+		(width 0.2)
+		(layer "F.Cu")
+		(net 6)
+	)
+	(segment
+		(start 128.851 76.679)
+		(end 128.851 72.450944)
+		(width 0.2)
+		(layer "F.Cu")
